File: v0p3/potentiostat_featherwing.kicad_pcb (KiCad board)
At the start: 2 copper layers, 22.9 x 50.8 mm, 20 parts, among them J1 Screw_Terminal_01x03, J2 Conn_01x03, J3 Conn_01x02, U1 feather_wing, U2 TS5A3160, U3 MCP6004

Commit message: Added gerbers, BOM and CPL for the four different ranges.
Other:
- board text added: "±10uA"
